File: hardware/bb-psu-mk-1.2.brd (EAGLE design)
At the start: 46 x 38 mm, 28 parts, among them IC1 LM317

Commit message: updates
Parts:
- removed OUT_PASS: M02PTH-CENTERED-R+, A_butts:1X02-CENTER-R+
- added R6: 330R, A_butts:RESISTOR-AXIAL-PTH-6.35MM
- PWR: value SWITCH-SPDTPTH-RA-2.54MM -> SWITCH-SPDTPTH-VERT-2.54MM; device A_butts:SPDT-RA-2.54MM -> A_butts:SWITCH-SPDT
- R1: value 5K -> 3k; device A_butts:RESISTOR-AXIAL-PTH-6.35MM -> A_butts:RESISTOR-AXIAL-PTH-7.62MM
- R2: value 8K2 -> 82k; device A_butts:RESISTOR-AXIAL-PTH-6.35MM -> A_butts:RESISTOR-AXIAL-PTH-7.62MM
- R3: value 15K -> 5K36; device A_butts:RESISTOR-AXIAL-PTH-6.35MM -> A_butts:RESISTOR-AXIAL-PTH-7.62MM
- R4: value 100K -> 10K2; device A_butts:3386U -> A_butts:RESISTOR-AXIAL-PTH-7.62MM
- R5: value 330R -> 100k; device A_butts:RESISTOR-AXIAL-PTH-6.35MM -> A_butts:3386U
- moved OUT_1 50.0 mm to (61.1, 14.7)
- moved U$1 46.9 mm to (59.5, 31.5)
- moved R5 31.0 mm to (41.0, 6.10)
- moved ON 15.5 mm to (20.7, 10.8), turned to 0 degrees
- moved PWR 11.1 mm to (48.5, 15.7), turned to 0 degrees
- moved C3 9.00 mm to (2.50, 17.2)
- moved TVS1 8.75 mm to (43.5, 17.5), turned to 90 degrees
- moved AMMETER 8.50 mm to (2.50, 23.8)
- moved F1 7.91 mm to (48.5, 26.5), turned to 270 degrees
- moved R4 7.28 mm to (33.5, 13.0), turned to 90 degrees
- moved C1 5.59 mm to (31.0, 22.5)
- moved C2 5.59 mm to (23.0, 22.5)
- moved OUT_2 4.50 mm to (17.0, 5.00)
- moved V_SEL 4.50 mm to (27.5, 3.70)
- moved IN_2 4.03 mm to (34.5, 36.0)
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Connections:
- removed net N$10: R2.P$1, V_SEL.P$2
- new net N$5: R4.P$1, V_SEL.P$3
- net GND: now also R4.P$2, R5.1; no longer OUT_PASS.1, R4.1
- net N$1: now also PWR.3; no longer F1.P$1
- net N$3: now also PWR.2; no longer PWR.1
- net N$4: now also R6.P$1; no longer R5.P$1
- net N$6: now also R2.P$1
- net N$7: now also V_SEL.P$2; no longer V_SEL.P$3
- net N$8: now also R5.3; no longer R4.3
- net VCC: now also R6.P$2; no longer R5.P$2
- net VIN: now also F1.P$1; no longer PWR.2
- net VOUT: no longer OUT_PASS.2
Routing:
- net VOUT: track 65.5 -> 0.00 mm
- net VIN: track 60.1 -> 0.00 mm
- net VCC: track 32.8 -> 0.00 mm
- net N$2: track 12.6 -> 0.00 mm
- net N$6: track 10.3 -> 0.00 mm
- net N$8: track 8.13 -> 0.00 mm
- net N$4: track 7.31 -> 0.00 mm
- net N$1: track 7.14 -> 0.00 mm
- net N$10: track 4.54 -> 0.00 mm
- net N$7: track 4.12 -> 0.00 mm
- net N$3: track 3.25 -> 0.00 mm
Other:
- board size 46 x 38 mm -> 51 x 38 mm
