File: hardware/bb-psu-mk-1.2.sch (EAGLE design)
At the start: 25 parts, among them IC1 LM317

Commit message: updates
Parts:
- removed OUT_PASS: M02PTH-CENTERED-R+, A_butts:M02PTH-CENTERED-R+
- added R6: 330R, A_butts:RESISTORPTH-AXIAL-6.35MM
- PWR: value SWITCH-SPDTPTH-RA-2.54MM -> SWITCH-SPDTPTH-VERT-2.54MM; device A_butts:SWITCH-SPDTPTH-RA-2.54MM -> A_butts:SWITCH-SPDTPTH-VERT-2.54MM
- R1: value 5K -> 3k; device A_butts:RESISTORPTH-AXIAL-6.35MM -> A_butts:RESISTORPTH-AXIAL-7.62MM
- R2: value 8K2 -> 82k; device A_butts:RESISTORPTH-AXIAL-6.35MM -> A_butts:RESISTORPTH-AXIAL-7.62MM
- R3: value 15K -> 5K36; device A_butts:RESISTORPTH-AXIAL-6.35MM -> A_butts:RESISTORPTH-AXIAL-7.62MM
- R4: value 100K -> 10K2; device A_butts:TRIMPOT-PTH-KNOB -> A_butts:RESISTORPTH-AXIAL-7.62MM
- R5: value 330R -> 100k; device A_butts:RESISTORPTH-AXIAL-6.35MM -> A_butts:TRIMPOT-PTH-KNOB
Connections:
- removed net N$10: R2.1, V_SEL.A
- new net N$5: R4.1, V_SEL.B
- net GND: now also R4.2, R5.CCW; no longer OUT_PASS.1, R4.CCW
- net N$1: now also PWR.NO; no longer F1.1
- net N$3: now also PWR.COM; no longer PWR.NC
- net N$4: now also R6.1; no longer R5.1
- net N$6: now also R2.1
- net N$7: now also V_SEL.A; no longer V_SEL.B
- net N$8: now also R5.CW; no longer R4.CW
- net VCC: now also R6.2; no longer R5.2
- net VIN: now also F1.1; no longer PWR.COM
- net VOUT: no longer OUT_PASS.2
Other:
- moved on the sheet: C1, C2, C3, D1, F1, IC1, ON, PWR, R1, R2, R3, TVS1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
